File: Clock_7Seg/Clock_7_Segment/Clock_7_Segment.kicad_pcb (KiCad board)
At the start: 2 copper layers, 100 x 100 mm, 46 parts, among them J1 Conn_01x06, J2 Conn_01x06, J3 Conn_01x03, U1 74HC595

Commit message: Add files via upload
First completed version
Parts:
- added D13: LED, LED_SMD:LED_0805_2012Metric_Pad1.15x1.40mm_HandSolder, F.Cu at (167.5, 91.0)
- added D14: LED, LED_SMD:LED_0805_2012Metric_Pad1.15x1.40mm_HandSolder, F.Cu at (167.5, 83.5)
- added D15: LED, LED_SMD:LED_0805_2012Metric_Pad1.15x1.40mm_HandSolder, F.Cu at (167.5, 107.0)
- added D16: LED, LED_SMD:LED_0805_2012Metric_Pad1.15x1.40mm_HandSolder, F.Cu at (167.5, 114.5)
- added D17: LED, LED_SMD:LED_0805_2012Metric_Pad1.15x1.40mm_HandSolder, F.Cu at (190.5, 91.0)
- added D18: LED, LED_SMD:LED_0805_2012Metric_Pad1.15x1.40mm_HandSolder, F.Cu at (190.5, 83.5)
- added D19: LED, LED_SMD:LED_0805_2012Metric_Pad1.15x1.40mm_HandSolder, F.Cu at (172.5, 99.0)
- added D20: LED, LED_SMD:LED_0805_2012Metric_Pad1.15x1.40mm_HandSolder, F.Cu at (185.5, 99.0)
- added D30: LED, LED_SMD:LED_0805_2012Metric_Pad1.15x1.40mm_HandSolder, F.Cu at (190.5, 107.0)
- added D31: LED, LED_SMD:LED_0805_2012Metric_Pad1.15x1.40mm_HandSolder, F.Cu at (190.5, 114.5)
- added D32: LED, LED_SMD:LED_0805_2012Metric_Pad1.15x1.40mm_HandSolder, F.Cu at (173.5, 118.5)
- added D33: LED, LED_SMD:LED_0805_2012Metric_Pad1.15x1.40mm_HandSolder, F.Cu at (184.0, 118.5)
- added D34: LED, LED_SMD:LED_0805_2012Metric_Pad1.15x1.40mm_HandSolder, F.Cu at (174.0, 80.0)
- added D35: LED, LED_SMD:LED_0805_2012Metric_Pad1.15x1.40mm_HandSolder, F.Cu at (184.5, 80.0)
- added D36: LED, LED_SMD:LED_0805_2012Metric_Pad1.15x1.40mm_HandSolder, F.Cu at (179.0, 126.0)
- added D37: LED, LED_SMD:LED_0805_2012Metric_Pad1.15x1.40mm_HandSolder, F.Cu at (179.0, 130.0)
- added D38: LED, LED_SMD:LED_0805_2012Metric_Pad1.15x1.40mm_HandSolder, F.Cu at (179.0, 158.0)
- added D39: LED, LED_SMD:LED_0805_2012Metric_Pad1.15x1.40mm_HandSolder, F.Cu at (179.0, 162.0)
- added J10: Conn_01x04, Connector_PinHeader_2.54mm:PinHeader_1x04_P2.54mm_Vertical, F.Cu at (209.0, 97.0)
- added J11: Conn_01x03, Connector_PinHeader_2.54mm:PinHeader_1x03_P2.54mm_Vertical, F.Cu at (197.0, 104.0)
- added J12: Conn_01x03, Connector_PinHeader_2.54mm:PinHeader_1x03_P2.54mm_Vertical, F.Cu at (208.0, 109.0)
- added J13: Conn_01x10, Connector_PinHeader_2.54mm:PinHeader_1x10_P2.54mm_Vertical, F.Cu at (210.0, 138.0)
- added J14: Conn_01x10, Connector_PinHeader_2.54mm:PinHeader_1x10_P2.54mm_Vertical, F.Cu at (196.7, 115.0)
- added J15: Conn_01x08, Connector_PinHeader_2.54mm:PinHeader_1x08_P2.54mm_Vertical, F.Cu at (210.0, 145.0)
- added J16: Conn_01x08, Connector_PinHeader_2.54mm:PinHeader_1x08_P2.54mm_Vertical, F.Cu at (196.7, 145.0)
- added J3: Conn_01x06, Connector_PinHeader_2.54mm:PinHeader_1x06_P2.54mm_Vertical, B.Cu at (172.5, 90.0)
- added J4: Conn_01x06, Connector_PinHeader_2.54mm:PinHeader_1x06_P2.54mm_Vertical, B.Cu at (172.5, 85.0)
- added J6: Conn_01x03, Connector_PinHeader_2.54mm:PinHeader_1x03_P2.54mm_Vertical, F.Cu at (176.5, 110.5)
- added J7: Conn_01x03, Connector_PinHeader_2.54mm:PinHeader_1x03_P2.54mm_Vertical, F.Cu at (179.0, 139.0)
- added J8: Conn_01x03, Connector_PinHeader_2.54mm:PinHeader_1x03_P2.54mm_Vertical, F.Cu at (197.0, 79.0)
- added J9: Conn_01x04, Connector_PinHeader_2.54mm:PinHeader_1x04_P2.54mm_Vertical, F.Cu at (197.0, 89.5)
- added Q1: S8550, Package_TO_SOT_SMD:SOT-23, F.Cu at (205.0, 82.0)
- added R13: R, Resistor_SMD:R_0805_2012Metric_Pad1.15x1.40mm_HandSolder, F.Cu at (167.5, 88.5)
- added R14: R, Resistor_SMD:R_0805_2012Metric_Pad1.15x1.40mm_HandSolder, F.Cu at (167.5, 86.0)
- added R15: R, Resistor_SMD:R_0805_2012Metric_Pad1.15x1.40mm_HandSolder, F.Cu at (167.5, 109.5)
- added R16: R, Resistor_SMD:R_0805_2012Metric_Pad1.15x1.40mm_HandSolder, F.Cu at (167.5, 112.0)
- added R17: R, Resistor_SMD:R_0805_2012Metric_Pad1.15x1.40mm_HandSolder, F.Cu at (190.5, 88.5)
- added R18: R, Resistor_SMD:R_0805_2012Metric_Pad1.15x1.40mm_HandSolder, F.Cu at (190.5, 86.0)
- added R19: R, Resistor_SMD:R_0805_2012Metric_Pad1.15x1.40mm_HandSolder, F.Cu at (176.5, 99.0)
- added R20: R, Resistor_SMD:R_0805_2012Metric_Pad1.15x1.40mm_HandSolder, F.Cu at (181.0, 99.0)
- added R30: R, Resistor_SMD:R_0805_2012Metric_Pad1.15x1.40mm_HandSolder, F.Cu at (190.5, 109.5)
- added R31: R, Resistor_SMD:R_0805_2012Metric_Pad1.15x1.40mm_HandSolder, F.Cu at (190.5, 112.0)
- added R32: R, Resistor_SMD:R_0805_2012Metric_Pad1.15x1.40mm_HandSolder, F.Cu at (177.0, 118.5)
- added R33: R, Resistor_SMD:R_0805_2012Metric_Pad1.15x1.40mm_HandSolder, F.Cu at (180.5, 118.5)
- added R34: R, Resistor_SMD:R_0805_2012Metric_Pad1.15x1.40mm_HandSolder, F.Cu at (177.5, 80.0)
- added R35: R, Resistor_SMD:R_0805_2012Metric_Pad1.15x1.40mm_HandSolder, F.Cu at (181.0, 80.0)
- added R36: R, Resistor_SMD:R_0805_2012Metric_Pad1.15x1.40mm_HandSolder, F.Cu at (174.0, 126.0)
- added R37: R, Resistor_SMD:R_0805_2012Metric_Pad1.15x1.40mm_HandSolder, F.Cu at (174.0, 130.0)
- added R38: R, Resistor_SMD:R_0805_2012Metric_Pad1.15x1.40mm_HandSolder, F.Cu at (174.0, 158.0)
- added R39: R, Resistor_SMD:R_0805_2012Metric_Pad1.15x1.40mm_HandSolder, F.Cu at (174.0, 162.0)
- added SW1: SW_DIP_x01, Button_Switch_THT:SW_PUSH_6mm_H4.3mm, F.Cu at (116.0, 168.0)
- added SW2: SW_DIP_x01, Button_Switch_THT:SW_PUSH_6mm_H4.3mm, F.Cu at (129.0, 168.0)
- added SW3: SW_DIP_x01, Button_Switch_THT:SW_PUSH_6mm_H4.3mm, F.Cu at (142.0, 168.0)
- added SW4: SW_DIP_x01, Button_Switch_THT:SW_PUSH_6mm_H4.3mm, F.Cu at (155.0, 168.0)
- added SW5: SW_DIP_x01, Button_Switch_THT:SW_PUSH_6mm_H4.3mm, F.Cu at (169.0, 168.0)
- added SW6: SW_DIP_x01, Button_Switch_THT:SW_PUSH_6mm_H4.3mm, F.Cu at (200.0, 168.0)
- added SW6: SW_DIP_x01, Button_Switch_THT:SW_PUSH_6mm_H4.3mm, F.Cu at (182.0, 168.0)
- added U2: 74HC595, Package_SO:SOIC-16_3.9x9.9mm_P1.27mm, B.Cu at (179.0, 99.5)
- added U3: LP2988-5.0_SOIC8_VSSOP8, Package_SO:SOIC-8-1EP_3.9x4.9mm_P1.27mm_EP2.95x4.9mm_Mask2.71x3.4mm, F.Cu at (203.0, 94.0)
- added U4: LMV601, Package_TO_SOT_SMD:SOT-363_SC-70-6, F.Cu at (203.0, 106.0)
- added U5: STM8S003F3P, Package_SO:TSSOP-20_4.4x6.5mm_P0.65mm, F.Cu at (203.4, 125.0)
- added U6: 74HC595, Package_SO:SOIC-16_3.9x9.9mm_P1.27mm, F.Cu at (203.2, 153.0)
- moved R27 87.8 mm to (126.0, 83.0), turned to 90 degrees
- moved R24 81.5 mm to (135.0, 159.0), turned to 270 degrees
- moved D24 77.6 mm to (132.0, 155.0), turned to 270 degrees
- moved R28 77.3 mm to (135.0, 83.0), turned to 90 degrees
- moved R4 74.7 mm to (122.0, 129.0), turned to 180 degrees
- moved R6 72.8 mm to (122.0, 145.0), turned to 180 degrees
- moved R29 72.3 mm to (143.0, 83.0), turned to 90 degrees
- moved R26 69.8 mm to (150.0, 159.0), turned to 270 degrees
- moved R5 69.3 mm to (122.0, 137.0), turned to 180 degrees
- moved D25 64.3 mm to (139.0, 155.0), turned to 270 degrees
- moved R25 63.6 mm to (142.0, 159.0), turned to 270 degrees
- moved D27 62.1 mm to (131.0, 86.0), turned to 90 degrees
- moved D8 60.9 mm to (153.0, 101.0)
- moved D5 60.8 mm to (125.0, 141.0), turned to 180 degrees
- moved D4 59.2 mm to (125.0, 133.0), turned to 180 degrees
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- renumbered D13 to D21, D14 to D22, D15 to D23, D16 to D24, D17 to D25, D18 to D26, D19 to D27, D20 to D28, D21 to D29, J3 to J5, R13 to R21, R14 to R22, R15 to R23, R16 to R24, R17 to R25, R18 to R26, R19 to R27, R20 to R28, R21 to R29
Routing:
- net G: track 0.00 -> 104.0 mm, vias 0 -> 4
- net CLR: track 0.00 -> 77.0 mm, vias 0 -> 4
- net OE: track 0.00 -> 75.2 mm, vias 0 -> 2
- net C: track 0.00 -> 65.8 mm, vias 0 -> 2
- net E: track 0.00 -> 61.4 mm, vias 0 -> 2
- net CLK: track 0.00 -> 60.4 mm, vias 0 -> 2
- net SER_IN: track 0.00 -> 49.1 mm, vias 0 -> 2
- net Ser_out: track 0.00 -> 48.7 mm, vias 0 -> 3
- net a: track 0.00 -> 47.1 mm, vias 0 -> 1
- net H_in: track 0.00 -> 42.7 mm
- net F: track 0.00 -> 42.1 mm
- net c: track 0.00 -> 36.7 mm, vias 0 -> 1
- net g: track 0.00 -> 34.0 mm, vias 0 -> 1
- net VCC: track 101.1 -> 67.2 mm
- net B: track 0.00 -> 33.9 mm, vias 0 -> 2
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- added copper zone on B.Cu, net GND
- added copper zone on F.Cu, net GND
- added copper zone on F.Cu, net Ground
- added copper zone on B.Cu, net gnd
- added copper zone on F.Cu, net gnd
Other:
- board text added: "CLR OE CLK SER IN GND VCC"
- board text added: "CLR OE CLK SER O GND VCC"
- board text added: "CLR OE CLK SER OUT GND VCC"
- board text added: "GND"
- board text added: "H input"
- board text added: "Not Conn"
- board text added: "VCC GND H"
