File: Clock_7Seg/Clock_7_Segment/Clock_7_Segment.sch (KiCad schematic (older format))
At the start: 46 parts, among them J1 Conn_01x06, J2 Conn_01x06, J3 Conn_01x03, U1 74HC595

Commit message: Add files via upload
First completed version
Parts:
- added D13, D14, D15, D16, D17, D18, D19, D20, D30, D31, D32, D33, D34, D35, D36, D37, D38, D39: LED, LED_SMD:LED_0805_2012Metric_Pad1.15x1.40mm_HandSolder, symbol Device:LED
- added J10, J9: Conn_01x04, Connector_PinHeader_2.54mm:PinHeader_1x04_P2.54mm_Vertical, symbol Connector_Generic:Conn_01x04
- added J11, J12, J6, J7, J8: Conn_01x03, Connector_PinHeader_2.54mm:PinHeader_1x03_P2.54mm_Vertical, symbol Connector_Generic:Conn_01x03
- added J13, J14: Conn_01x10, Connector_PinHeader_2.54mm:PinHeader_1x10_P2.54mm_Vertical, symbol Connector_Generic:Conn_01x10
- added J15, J16: Conn_01x08, Connector_PinHeader_2.54mm:PinHeader_1x08_P2.54mm_Vertical, symbol Connector_Generic:Conn_01x08
- added J3, J4: Conn_01x06, Connector_PinHeader_2.54mm:PinHeader_1x06_P2.54mm_Vertical, symbol Connector_Generic:Conn_01x06
- added Q1: S8550, Package_TO_SOT_SMD:SOT-23, symbol Transistor_BJT:S8550
- added R13, R14, R15, R16, R17, R18, R19, R20, R30, R31, R32, R33, R34, R35, R36, R37, R38, R39: R, Resistor_SMD:R_0805_2012Metric_Pad1.15x1.40mm_HandSolder, symbol Device:R
- added SW1, SW2, SW3, SW4, SW5, SW6: SW_DIP_x01, Button_Switch_THT:SW_PUSH_6mm_H4.3mm, symbol Switch:SW_DIP_x01
- added U2, U6: 74HC595, Package_SO:SOIC-16_3.9x9.9mm_P1.27mm, symbol 74xx:74HC595
- added U3: LP2988-5.0_SOIC8_VSSOP8, Package_SO:SOIC-8-1EP_3.9x4.9mm_P1.27mm_EP2.95x4.9mm_Mask2.71x3.4mm, symbol Regulator_Linear:LP2988-5.0_SOIC8_VSSOP8
- added U4: LMV601, Package_TO_SOT_SMD:SOT-363_SC-70-6, symbol Amplifier_Operational:LMV601
- added U5: STM8S003F3P, Package_SO:TSSOP-20_4.4x6.5mm_P0.65mm, symbol MCU_ST_STM8:STM8S003F3P
- renumbered D13 to D21, D14 to D22, D15 to D23, D16 to D24, D17 to D25, D18 to D26, D19 to D27, D20 to D28, D21 to D29, J3 to J5, R13 to R21, R14 to R22, R15 to R23, R16 to R24, R17 to R25, R18 to R26, R19 to R27, R20 to R28, R21 to R29
Connections:
- new net: D13.2 (A), R13.1
- new net: D14.2 (A), R14.1
- new net: D15.2 (A), R15.1
- new net: D16.2 (A), R16.1
- new net: D17.2 (A), R17.1
- new net: D18.2 (A), R18.1
- new net: D19.2 (A), R19.1
- new net: D20.2 (A), R20.1
- new net: D30.2 (A), R30.1
- new net: D31.2 (A), R31.1
- new net: D32.2 (A), R32.1
- new net: D33.2 (A), R33.1
- new net: D34.2 (A), R34.1
- new net: D35.2 (A), R35.1
- new net: D36.2 (A), R36.1
- new net: D37.2 (A), R37.1
- new net: D38.2 (A), R38.1
- new net: D39.2 (A), R39.1
- new net: J8.1 (Pin_1), Q1.1 (E)
- new net: J8.2 (Pin_2), Q1.2 (B)
- new net: J8.3 (Pin_3), Q1.3 (C)
- new net: J10.1 (Pin_1), U3.1 (BP)
- new net: J10.2 (Pin_2), U3.2 (DELAY)
- new net: J10.3 (Pin_3), U3.3 (GND)
- new net: J10.4 (Pin_4), U3.4 (IN)
- new net: J9.1 (Pin_1), U3.5 (OUT)
- new net: J9.2 (Pin_2), U3.6 (SENSE)
- new net: J9.3 (Pin_3), U3.7 (~ERROR)
- new net: J11.1 (Pin_1), U4.1 (+)
- new net: J11.2 (Pin_2), U4.2 (V-)
- new net: J11.3 (Pin_3), U4.3 (-)
- new net: J12.1 (Pin_1), U4.4
- new net: J12.2 (Pin_2), U4.5 (~SHDN)
- new net: J12.3 (Pin_3), U4.6 (V+)
- new net: J14.1 (Pin_1), U5.1 (PD4)
- new net: J13.1 (Pin_1), U5.11 (PB5)
- new net: J13.2 (Pin_2), U5.12 (PB4)
- new net: J13.3 (Pin_3), U5.13 (PC3)
- new net: J13.4 (Pin_4), U5.14 (PC4)
- new net: J13.5 (Pin_5), U5.15 (PC5)
- new net: J13.6 (Pin_6), U5.16 (PC6)
- new net: J13.7 (Pin_7), U5.17 (PC7)
- new net: J14.2 (Pin_2), U5.2 (PD5)
- new net: J14.3 (Pin_3), U5.3 (PD6)
- new net: J16.1 (Pin_1), U6.1 (QB)
- new net: J15.7 (Pin_7), U6.10 (~SRCLR)
- new net: J15.6 (Pin_6), U6.11 (SRCLK)
- new net: J15.5 (Pin_5), U6.12 (RCLK)
- new net: J15.4 (Pin_4), U6.13 (~OE)
- new net: J15.3 (Pin_3), U6.14 (SER)
- new net: J15.2 (Pin_2), U6.15 (QA)
- new net: J15.1 (Pin_1), U6.16 (VCC)
- new net: J16.2 (Pin_2), U6.2 (QC)
- new net: J16.3 (Pin_3), U6.3 (QD)
- new net: J16.4 (Pin_4), U6.4 (QE)
- new net: J16.5 (Pin_5), U6.5 (QF)
- new net: J16.6 (Pin_6), U6.6 (QG)
- new net: J16.7 (Pin_7), U6.7 (QH)
- new net: J16.8 (Pin_8), U6.8 (GND)
- new net: J15.8 (Pin_8), U6.9 (QH')
- new net 8: J9.4 (Pin_4), U3.8 (~SHTD)
- new net Ground: D36.1 (K), D37.1 (K), D38.1 (K), D39.1 (K), J7.2 (Pin_2)
- new net H_in: J7.3 (Pin_3), R36.2, R37.2, R38.2, R39.2
- new net a: R13.2, R14.2, U2.15 (QA)
- new net b: R15.2, R16.2, U2.1 (QB)
- new net c: R17.2, R18.2, U2.2 (QC)
- new net c10: J14.10 (Pin_10), U5.10 (PA3)
- new net c18: J13.8 (Pin_8), U5.18 (PD1)
- new net c19: J13.9 (Pin_9), U5.19 (PD2)
- new net c20: J13.10 (Pin_10), U5.20 (PD3)
- new net c4: J14.4 (Pin_4), U5.4 (NRST)
- new net c5: J14.5 (Pin_5), U5.5 (PA1)
- new net c6: J14.6 (Pin_6), U5.6 (PA2)
- new net c7: J14.7 (Pin_7), U5.7 (VSS)
- new net c8: J14.8 (Pin_8), U5.8 (VCAP)
- new net c9: J14.9 (Pin_9), U5.9 (VDD)
- new net clk: J3.3 (Pin_3), J4.3 (Pin_3), U2.11 (SRCLK), U2.12 (RCLK)
- new net clr: J3.1 (Pin_1), J4.1 (Pin_1), U2.10 (~SRCLR)
- new net d: R19.2, R20.2, U2.3 (QD)
- new net e: R30.2, R31.2, U2.4 (QE)
- new net f: R32.2, R33.2, U2.5 (QF)
- new net g: R34.2, R35.2, U2.6 (QG)
- new net gnd: D13.1 (K), D14.1 (K), D15.1 (K), D16.1 (K), D17.1 (K), D18.1 (K), D19.1 (K), D20.1 (K), D30.1 (K), D31.1 (K), D32.1 (K), D33.1 (K), D34.1 (K), D35.1 (K), J3.5 (Pin_5), J4.5 (Pin_5), J6.2 (Pin_2), U2.8 (GND)
- new net h: J6.3 (Pin_3), U2.7 (QH)
- new net oe: J3.2 (Pin_2), J4.2 (Pin_2), U2.13 (~OE)
- new net ser_in: J3.4 (Pin_4), U2.14 (SER)
- new net ser_out: J4.4 (Pin_4), U2.9 (QH')
- new net vcc: J3.6 (Pin_6), J4.6 (Pin_6), J6.1 (Pin_1), U2.16 (VCC)
- no-connect marks 0 -> 1
Other:
- note added: "BIG SEVEN SEGMENT COMPONENT"
- note added: "Dot display"
- note added: "SMALL SEVEN SEGMENT COMPONENT"
- note added: "SOT-23"
- note added: "SOT-363"
- note added: "switch interface\n"
- note removed: "SEVEN SEGMENT COMPONENT"
